File: transistors/slides-handouts/ohms-law-1.sch (EAGLE design)
At the start: 15 parts

Commit message: updated
Parts:
- R11: value 1k -> 3000 ohms "orange black red"
- R12: value 1k -> 1000 ohms "brown black red"
- R2: value 1000 ohms "brown black red" -> 1500 ohms "brown green red"
- R5: value 1000 ohms "brown black red" -> 2000 ohms "red black red"
- R6: value 1000 ohms "brown black red" -> 10 ohms "brown black black"
- R7: value 1000 ohms "brown black red" -> 20 ohms "red black black"
Other:
- note added: "0 VOLTS HERE"
- note added: "15 VOLTS HERE"
- note added: "<-- AMPS THROUGH HERE?"
- note added: "Copyright (c) 2017 Durham Makerspace - Licensed under Creative Commons CC0 1.0 Universal"
- note removed: "* CONVENTIONAL CURRENT FLOW USED THROUGHOUT"
- moved on the sheet: G1, G2, G3, R11, R12, R3, R4, R5
