File: transistors/wiring/common-emitter-1.sch (EAGLE design)
At the start: 9 parts, among them T1 2N3904

Commit message: initial draft
Parts:
- R1: value 100k "104" -> 1k "102"
- R2: value 1k "brn blk red" -> 100k "brn blk ylw"
Changed lines of the file:
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@@
 <part name="FRAME1" library="frames" deviceset="LETTER_L" device=""/>
 <part name="R3" library="rcl" deviceset="R-US_" device="0309/12" value="10k &quot;brn blk org&quot;"/>
-<part name="R2" library="rcl" deviceset="R-US_" device="0309/12" value="1k &quot;brn blk red&quot;"/>
-<part name="R1" library="SparkFun-Retired" deviceset="TRIMPOT" device="3362U-2" value="100k &quot;104&quot;"/>
+<part name="R2" library="rcl" deviceset="R-US_" device="0309/12" value="100k &quot;brn blk ylw&quot;"/>
+<part name="R1" library="SparkFun-Retired" deviceset="TRIMPOT" device="3362U-2" value="1k &quot;102&quot;"/>
 <part name="BT1" library="SparkFun-Batteries" deviceset="BATTERY" device="-AAA_KIT"/>
 <part name="TP1" library="SparkFun-Connectors" deviceset="TEST-POINT" device="2" value="TEST-POINT1"/>

Commit message: updates
Parts:
- ..: value BLACK DMM LEAD HERE -> BLACK/COMMON METER LEAD HERE
- BT1: value (none) -> 4.5 Volts
- R1: value 1k "102" -> 1000 "102"
- R2: value 100k "brn blk ylw" -> 1000000 "brn blk grn"
- R3: value 10k "brn blk org" -> 10000 "brn blk org"
- renumbered BATTERY_POSITIVE to ., GROUND to ..
Connections:
- new net N$7: BT1.+
- net N$4: no longer BT1.+
Other:
- note added: "0.61"
- note added: "<-- Disconnect here to save battery"
- note added: "Black wire"
- note added: "Current Event Workshops"
- note added: "Pete Soper - Durham Makerspace"
- note added: "Red wire from battery holder"
- note added: "Simple amplifier operation. As R1 is adjusted test point 2 voltage goes from the supply rail toward ground as the transistor is turned on."
- note added: "https://github.com/splatspace/currentevent"
- note removed: ""BLACK/BLUE BREADBOARD ROW OF HOLES""
- note removed: ""RED BREADBOARD ROW OF HOLES""
- note removed: "0.50"
- note removed: "Current Event Intro to Transistors Part 1"
- moved on the sheet: BT1, R1, R2, TP1, TP2
