File: transistors/wiring/common-collector-1.sch (EAGLE design)
At the start: 14 parts, among them M1 MOTOR10MM, Q1 60V/32A/35mΩ, T1 2N3904

Commit message: back to one page
Parts:
- removed D2: DIODE-1N4148, SparkFun-DiscreteSemi:DIODE-1N4148
- removed M1: MOTOR10MM, SparkFun-Electromechanical:MOTOR10MM
- removed Q1: 60V/32A/35mΩ, SparkFun-DiscreteSemi:MOSFET-NCH-FQP30N06L
- removed R4: 1m "brn blk grn", rcl:R-US_0309/12
Connections:
- removed net +12V: D2.C, M1.+
- removed net N$10: Q1.S
- removed net N$12: D2.A, M1.-, Q1.D
- removed net N$13: Q1.G
Changed lines of the file:
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@@
 <part name="FRAME1" library="PJS" deviceset="LETTER_L" device=""/>
 <part name="D1" library="SparkFun-LED" deviceset="LED" device="5MM" value="COLOR"/>
-<part name="Q1" library="SparkFun-DiscreteSemi" deviceset="MOSFET-NCH" device="-FQP30N06L" value="60V/32A/35mΩ"/>
-<part name="M1" library="SparkFun-Electromechanical" deviceset="MOTOR" device="10MM"/>
-<part name="P+1" library="supply1" deviceset="+12V" device=""/>
-<part name="D2" library="SparkFun-DiscreteSemi" deviceset="DIODE" device="-1N4148" value=""/>
-<part name="R4" library="rcl" deviceset="R-US_" device="0309/12" value="1m &quot;brn blk grn&quot;"/>
 </parts>
 <sheets>
@@
 <instance part="FRAME1" gate="G$2" x="17.78" y="-93.98"/>
 <instance part="D1" gate="G$1" x="22.86" y="-20.32"/>
-<instance part="Q1" gate="NMOS" x="256.54" y="-5.08"/>
-<instance part="M1" gate="G$1" x="259.08" y="20.32"/>
-<instance part="P+1" gate="1" x="259.08" y="50.8"/>
-<instance part="D2" gate="G$1" x="281.94" y="20.32" rot="R90"/>
-<instance part="R4" gate="G$1" x="236.22" y="-15.24" smashed="yes" rot="R270">
-<attribute name="NAME" x="242.57" y="-16.7386" size="1.778" layer="95" rot="R180"/>
-<attribute name="VALUE" x="242.57" y="-13.462" size="1.778" layer="96"/>
-</instance>
 </instances>
 <busses>
@@
 </segment>
 </net>
-<net name="N$10" class="0">
-<segment>
-<pinref part="Q1" gate="NMOS" pin="S"/>
-<wire x1="259.08" y1="-10.16" x2="259.08" y2="-22.86" width="0.1524" layer="91"/>
-</segment>
-</net>
-<net name="+12V" class="0">
-<segment>
-<pinref part="P+1" gate="1" pin="+12V"/>
-<pinref part="M1" gate="G$1" pin="+"/>
-<wire x1="259.08" y1="48.26" x2="259.08" y2="30.48" width="0.1524" layer="91"/>
-<pinref part="D2" gate="G$1" pin="C"/>
-<wire x1="259.08" y1="30.48" x2="259.08" y2="25.4" width="0.1524" layer="91"/>
-<wire x1="281.94" y1="22.86" x2="281.94" y2="30.48" width="0.1524" layer="91"/>
-<wire x1="281.94" y1="30.48" x2="259.08" y2="30.48" width="0.1524" layer="91"/>
-<junction x="259.08" y="30.48"/>
-</segment>
-</net>
-<net name="N$12" class="0">
-<segment>
-<pinref part="M1" gate="G$1" pin="-"/>
-<pinref part="Q1" gate="NMOS" pin="D"/>
-<wire x1="259.08" y1="15.24" x2="259.08" y2="7.62" width="0.1524" layer="91"/>
-<pinref part="D2" gate="G$1" pin="A"/>
-<wire x1="259.08" y1="7.62" x2="259.08" y2="0" width="0.1524" layer="91"/>
-<wire x1="281.94" y1="17.78" x2="281.94" y2="7.62" width="0.1524" layer="91"/>
-<wire x1="281.94" y1="7.62" x2="259.08" y2="7.62" width="0.1524" layer="91"/>
-<junction x="259.08" y="7.62"/>
-</segment>
-</net>
-<net name="N$13" class="0">
-<segment>
-<pinref part="Q1" gate="NMOS" pin="G"/>
-<wire x1="220.98" y1="-7.62" x2="251.46" y2="-7.62" width="0.1524" layer="91"/>
-</segment>
-</net>
